File: matrix.kicad_sch (KiCad schematic)
At the start: 204 parts, among them SW10 MX_Keyswitch, SW100 MX_Keyswitch, SW101 MX_Keyswitch, SW102 MX_Keyswitch, SW103 MX_Keyswitch, SW104 MX_Keyswitch, SW11 MX_Keyswitch, SW12 MX_Keyswitch, SW13 MX_Keyswitch, SW14 MX_Keyswitch, SW15 MX_Keyswitch, SW16 MX_Keyswitch, SW17 MX_Keyswitch, SW18 MX_Keyswitch, SW19 MX_Keyswitch, SW20 MX_Keyswitch, SW21 MX_Keyswitch, SW22 MX_Keyswitch, SW23 MX_Keyswitch, SW24 MX_Keyswitch, SW25 MX_Keyswitch, SW26 MX_Keyswitch, SW27 MX_Keyswitch, SW28 MX_Keyswitch, SW29 MX_Keyswitch, SW3 MX_Keyswitch, SW30 MX_Keyswitch, SW31 MX_Keyswitch, SW32 MX_Keyswitch, SW33 MX_Keyswitch, SW34 MX_Keyswitch, SW35 MX_Keyswitch, SW36 MX_Keyswitch, SW37 MX_Keyswitch, SW38 MX_Keyswitch, SW39 MX_Keyswitch, SW4 MX_Keyswitch, SW40 MX_Keyswitch, SW41 MX_Keyswitch, SW42 MX_Keyswitch, SW43 MX_Keyswitch, SW44 MX_Keyswitch, SW45 MX_Keyswitch, SW46 MX_Keyswitch, SW47 MX_Keyswitch, SW48 MX_Keyswitch, SW49 MX_Keyswitch, SW5 MX_Keyswitch, SW50 MX_Keyswitch, SW51 MX_Keyswitch, SW52 MX_Keyswitch, SW53 MX_Keyswitch, SW54 MX_Keyswitch, SW55 MX_Keyswitch, SW56 MX_Keyswitch, SW57 MX_Keyswitch, SW58 MX_Keyswitch, SW59 MX_Keyswitch, SW6 MX_Keyswitch, SW60 MX_Keyswitch, SW61 MX_Keyswitch, SW62 MX_Keyswitch, SW63 MX_Keyswitch, SW64 MX_Keyswitch, SW65 MX_Keyswitch, SW66 MX_Keyswitch, SW67 MX_Keyswitch, SW68 MX_Keyswitch, SW69 MX_Keyswitch, SW7 MX_Keyswitch, SW70 MX_Keyswitch, SW71 MX_Keyswitch, SW72 MX_Keyswitch, SW73 MX_Keyswitch, SW74 MX_Keyswitch, SW75 MX_Keyswitch, SW76 MX_Keyswitch, SW77 MX_Keyswitch, SW78 MX_Keyswitch, SW79 MX_Keyswitch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

Commit message: MCU/USB/Switch Matrix Schematics
Parts:
- removed D100, D101, D102, D72, D78, D82, D83, D84, D88, D89, D90, D94, D95, D96, D97: 1N4148W, symbol Device:D
- removed SW102, SW103, SW104, SW74, SW80, SW84, SW85, SW86, SW90, SW91, SW92, SW96, SW97, SW98, SW99: MX_Keyswitch, symbol Switch:SW_Push

Commit message: Footprints
Parts:
- D1, D10, D11, D12, D13, D14, D15, D16, D17, D18, D19, D2, D20, D21, D22, D23, D24, D25, D26, D27, D28, D29, D3, D30, D31, D32, D33, D34, D35, D36, D37, D38, D39, D4, D40, D41, D42, D43, D44, D45, D46, D47, D48, D49, D5, D50, D51, D52, D53, D54, D55, D56, D57, D58, D59, D6, D60, D61, D62, D63, D64, D65, D66, D67, D68, D69, D7, D70, D71, D73, D74, D75, D76, D77, D79, D8, D80, D81, D85, D86, D87, D9, D91, D92, D93, D98, D99: footprint (none) -> Diode_SMD:D_SOD-123
- SW10, SW100, SW101, SW11, SW12, SW13, SW14, SW15, SW16, SW17, SW18, SW21, SW22, SW23, SW24, SW25, SW26, SW27, SW28, SW29, SW3, SW30, SW31, SW32, SW33, SW34, SW37, SW39, SW4, SW41, SW43, SW45, SW47, SW49, SW5, SW51, SW52, SW53, SW54, SW55, SW56, SW57, SW58, SW59, SW6, SW60, SW61, SW62, SW63, SW64, SW65, SW66, SW67, SW68, SW69, SW7, SW70, SW71, SW72, SW75, SW76, SW77, SW79, SW8, SW81, SW87, SW88, SW89, SW9, SW93, SW94, SW95: footprint (none) -> MX_Hotswap:MX-Hotswap-1U
- SW19, SW83: footprint (none) -> MX_Hotswap:MX-Hotswap-1.5U
- SW20: footprint (none) -> MX_Hotswap:MX-Hotswap-1.75U
- SW35, SW78: footprint (none) -> MX_Hotswap:MX-Hotswap-2.25U
- SW36, SW38, SW40, SW44, SW46, SW48, SW50: footprint (none) -> MX_Hotswap:MX-Hotswap-1.25U
- SW42: footprint (none) -> MX_Hotswap:MX-Hotswap-6.25U
- SW73: footprint (none) -> MX_Hotswap:MX-Hotswap-2.75U
- SW82: footprint (none) -> MX_Hotswap:MX-Hotswap-2U

Commit message: Putting diodes in their place
Parts:
- SW10, SW100, SW101, SW11, SW12, SW13, SW14, SW15, SW16, SW17, SW18, SW21, SW22, SW23, SW24, SW25, SW26, SW27, SW28, SW29, SW3, SW30, SW31, SW32, SW33, SW34, SW37, SW39, SW4, SW41, SW43, SW45, SW47, SW49, SW5, SW51, SW52, SW53, SW54, SW55, SW56, SW57, SW58, SW59, SW6, SW60, SW61, SW62, SW63, SW64, SW65, SW66, SW67, SW68, SW69, SW7, SW70, SW71, SW72, SW75, SW76, SW77, SW79, SW8, SW81, SW87, SW88, SW89, SW9, SW93, SW94, SW95: footprint MX_Hotswap:MX-Hotswap-1U -> MX_Solderable:MX-Solderable-1U
- SW19, SW83: footprint MX_Hotswap:MX-Hotswap-1.5U -> MX_Solderable:MX-Solderable-1.5U
- SW20: footprint MX_Hotswap:MX-Hotswap-1.75U -> MX_Solderable:MX-Solderable-1.75U
- SW35, SW78: footprint MX_Hotswap:MX-Hotswap-2.25U -> MX_Solderable:MX-Solderable-2.25U
- SW36, SW38, SW40, SW44, SW46, SW48, SW50: footprint MX_Hotswap:MX-Hotswap-1.25U -> MX_Solderable:MX-Solderable-1.25U
- SW42: footprint MX_Hotswap:MX-Hotswap-6.25U -> MX_Solderable:MX-Solderable-6.25U
- SW73: footprint MX_Hotswap:MX-Hotswap-2.75U -> MX_Solderable:MX-Solderable-2.75U
- SW82: footprint MX_Hotswap:MX-Hotswap-2U -> MX_Solderable:MX-Solderable-2U
